File: PCB/DMX_ControllerBoard/DMX_ControllerBoard.kicad_pcb (KiCad board)
At the start: 4 copper layers, 100 x 36.8 mm, 42 parts, among them J1 Screw_Terminal_01x03, J2 Screw_Terminal_01x03, J3 PWR_IN, J4 Screw_Terminal_01x03, J5 Conn_Left, J6 Screw_Terminal_01x03, J7 ProgrammingHeader, SW1 SW_SPST, SW2 SW_SPST, SW3 SW_SPST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

Commit message: Started work on finding power problems with original board and testing a new ESP32 board
Parts:
- removed TP1, TP2: TP_5V, TestPoint:TestPoint_2Pads_Pitch2.54mm_Drill0.8mm
- removed U3: H7233-1, Package_TO_SOT_SMD:SOT-89-3_Handsoldering
- added C2: 10uF/25V, Capacitor_SMD:C_0805_2012Metric, F.Cu at (62.1, 25.9)
- added C5: 1uF/10V, Capacitor_SMD:C_0805_2012Metric, F.Cu at (71.0, 35.7)
- added C6: 100uF/6.3V, Capacitor_SMD:C_1206_3216Metric, F.Cu at (68.6, 35.7)
- added U1: AMS1117-3.3, Package_TO_SOT_SMD:SOT-223-3_TabPin2, F.Cu at (61.1, 31.5)
- C1: value 100nF -> 10uF/25V; footprint Capacitor_SMD:C_0805_2012Metric_Pad1.18x1.45mm_HandSolder -> Capacitor_SMD:C_0805_2012Metric
- C3: value 1uF -> 100nF/16V; footprint Capacitor_SMD:C_0805_2012Metric_Pad1.18x1.45mm_HandSolder -> Capacitor_SMD:C_0805_2012Metric
- C4: value 1uF -> 22uF/25V; footprint Capacitor_SMD:C_0805_2012Metric_Pad1.18x1.45mm_HandSolder -> Capacitor_SMD:C_0805_2012Metric
- moved C3 13.6 mm to (73.3, 35.7), turned to -90 degrees
- moved C4 8.95 mm to (62.1, 23.7)
- moved C1 1.30 mm to (61.2, 37.2), turned to 180 degrees
Connections:
- C1 pad 1: GND -> +5V
- C1 pad 2: +3V3 -> GND
- C3 pad 1: GND -> +3V3
- C3 pad 2: +5V -> GND
- J7 pad 1: Net-(J7-Pad1) -> unconnected-(J7-Pad1)
- J7 pad 5: Net-(J7-Pad5) -> unconnected-(J7-Pad5)
- U2 pad 1: Net-(U2-Pad1) -> unconnected-(U2-Pad1)
- U4 pad 1: Net-(U4-Pad1) -> unconnected-(U4-Pad1)
- U4 pad 2: Net-(U4-Pad2) -> unconnected-(U4-Pad2)
- U4 pad 3: Net-(U4-Pad3) -> unconnected-(U4-Pad3)
- U8 pad 10: Net-(U8-Pad10) -> unconnected-(U8-Pad10)
- U8 pad 11: Net-(U8-Pad11) -> unconnected-(U8-Pad11)
- U8 pad 13: Net-(U8-Pad13) -> unconnected-(U8-Pad13)
- U8 pad 14: Net-(U8-Pad14) -> unconnected-(U8-Pad14)
- U8 pad 2: Net-(U8-Pad2) -> unconnected-(U8-Pad2)
- U8 pad 4: Net-(U8-Pad4) -> unconnected-(U8-Pad4)
- U8 pad 9: Net-(U8-Pad9) -> unconnected-(U8-Pad9)
Routing:
- net +5V: track 26.4 -> 21.2 mm, vias 3 -> 4
- net GND: track 44.2 -> 48.0 mm, vias 28 -> 24
- net +3V3: track 91.9 -> 94.6 mm
Other:
- net class Default removed
- board text removed: "+3.3V | GND"
- board text removed: "+5V | GND"

Commit message: Added more labeling to ESP32 board
Connections:
- J7 pad 1: unconnected-(J7-Pad1) -> BOOT_MODE
- J7 pad 5: unconnected-(J7-Pad5) -> RESET
Routing:
- net RESET: track 12.6 -> 48.1 mm, vias 0 -> 1
- net BOOT_MODE: track 7.66 -> 15.0 mm, vias 0 -> 1

Commit message: Initial commit of ESP32 based PCB
Parts:
- removed R11, R12, R13: 10k, Resistor_SMD:R_0805_2012Metric_Pad1.20x1.40mm_HandSolder
- added R6: 10k, Resistor_SMD:R_0805_2012Metric_Pad1.20x1.40mm_HandSolder, F.Cu at (71.9, 41.1)
- added U3: 74LVC2T45DC, Package_SO:VSSOP-8_2.3x2mm_P0.5mm, F.Cu at (69.3, 41.5)
- added U5: 74LVC2T45DC, Package_SO:VSSOP-8_2.3x2mm_P0.5mm, F.Cu at (82.2, 41.5)
- moved R10 31.4 mm to (84.6, 41.1), turned to -90 degrees
- moved J6 6.00 mm to (89.8, 50.7)
- moved J4 4.00 mm to (74.5, 50.7)
- moved J2 2.00 mm to (59.3, 50.7)
Connections:
- J1 pad 3: B1 -> Button1_sense
- J2 pad 3: B2 -> Button2_sense
- J4 pad 3: B3 -> Button3_sense
- J6 pad 3: B4 -> Button4_sense
- R10 pad 1: B1 -> Net-(R10-Pad1)
- R10 pad 2: GND -> +5V
- U8 pad 12: B4 -> unconnected-(U8-Pad12)
- U8 pad 2: unconnected-(U8-Pad2) -> B4
Routing:
- net B1: track 43.2 -> 15.7 mm
- net Button4_sense: track 0.00 -> 23.1 mm
- net Button1_sense: track 0.00 -> 18.4 mm
- net +3V3: track 94.6 -> 111.7 mm
- net B3: track 30.9 -> 21.9 mm
- net Button3_sense: track 0.00 -> 8.84 mm
- net B2: track 32.6 -> 24.0 mm
- net B4: track 32.4 -> 24.3 mm, vias 0 -> 2
- net Button2_sense: track 0.00 -> 7.71 mm
- net +5V: track 21.2 -> 26.4 mm, vias 4 -> 8
- net GND: track 48.0 -> 44.0 mm, vias 24 -> 22
- net Net-(R6-Pad1): track 0.00 -> 1.86 mm
- net Net-(R10-Pad1): track 0.00 -> 1.73 mm
