File: PCB/DMX_ControllerBoard/DMX_ControllerBoard.kicad_sch (KiCad schematic)
At the start: 43 parts, among them J1 Screw_Terminal_01x03, J2 Screw_Terminal_01x03, J3 PWR_IN, J4 Screw_Terminal_01x03, J5 Conn_Left, J6 Screw_Terminal_01x03, J7 ProgrammingHeader, SW1 SW_SPST, SW2 SW_SPST, SW3 SW_SPST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

Commit message: Added more labeling to ESP32 board
Connections:
- net BOOT_MODE: now also J7.1 (Pin_1)
- net RESET: now also J7.5 (Pin_5)
- no-connect marks 13 -> 11
Changed lines of the file:
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@@
   (no_connect (at 59.69 179.07))
   (no_connect (at 54.61 179.07))
-  (no_connect (at 82.55 118.11))
   (no_connect (at 130.81 29.21))
   (no_connect (at 29.21 63.5))
@@
   (no_connect (at 29.21 55.88))
   (no_connect (at 59.69 63.5))
-  (no_connect (at 82.55 128.27))
   (no_connect (at 29.21 66.04))
   (wire (pts (xy 128.27 33.02) (xy 128.27 34.29))
@@
     )
   )
+  (global_label "RESET" (shape input) (at 82.55 128.27 180) (fields_autoplaced)
+    (effects (font (size 1.27 1.27)) (justify right))
+    (property "Intersheet References" "${INTERSHEET_REFS}" (id 0) (at 53.34 90.17 0)
+      (effects (font (size 1.27 1.27)) hide)
+    )
+  )
   (global_label "RESET" (shape input) (at 29.21 38.1 180) (fields_autoplaced)
     (effects (font (size 1.27 1.27)) (justify right))
@@
     (effects (font (size 1.27 1.27)) (justify left))
     (property "Intersheet References" "${INTERSHEET_REFS}" (id 0) (at 0 0 0)
+      (effects (font (size 1.27 1.27)) hide)
+    )
+  )
+  (global_label "BOOT_MODE" (shape input) (at 82.55 118.11 180) (fields_autoplaced)
+    (effects (font (size 1.27 1.27)) (justify right))
+    (property "Intersheet References" "${INTERSHEET_REFS}" (id 0) (at 142.24 156.21 0)
       (effects (font (size 1.27 1.27)) hide)
     )
@@
   (symbol (lib_id "power:PWR_FLAG") (at 21.59 173.99 0) (unit 1)
     (in_bom yes) (on_board yes)
-    (property "Reference" "" (id 0) (at 21.59 172.085 0)
+    (property "Reference" "#FLG0102" (id 0) (at 21.59 172.085 0)
       (effects (font (size 1.27 1.27)) hide)
     )
@@
   (symbol (lib_id "power:PWR_FLAG") (at 21.59 176.53 180) (unit 1)
     (in_bom yes) (on_board yes)
-    (property "Reference" "" (id 0) (at 21.59 178.435 0)
+    (property "Reference" "#FLG0103" (id 0) (at 21.59 178.435 0)
       (effects (font (size 1.27 1.27)) hide)
     )
@@
   (symbol (lib_id "power:PWR_FLAG") (at 91.44 168.91 0) (unit 1)
     (in_bom yes) (on_board yes)
-    (property "Reference" "" (id 0) (at 91.44 167.005 0)
-      (effects (font (size 1.27 1.27)) hide)
-    )
+    (property "Reference" "#FLG0101" (id 0) (at 91.44 167.005 0)
+      (effects (font (size 1.27 1.27)) hide)
+    )

Commit message: Initial commit of ESP32 based PCB
Parts:
- removed R11, R12, R13: 10k, Resistor_SMD:R_0805_2012Metric_Pad1.20x1.40mm_HandSolder, symbol Device:R_Small
- added R6: 10k, Resistor_SMD:R_0805_2012Metric_Pad1.20x1.40mm_HandSolder, symbol Device:R_Small
- added U3, U5: 74LVC2T45DC, Package_SO:VSSOP-8_2.3x2mm_P0.5mm, symbol Logic_LevelTranslator:74LVC2T45DC
Connections:
- net +3V3: now also U3.8 (VCCB), U5.8 (VCCB)
- net +5V: now also R10.2, R6.2, U3.1 (VCCA), U5.1 (VCCA)
- net B1: now also U3.7 (1B); no longer J1.3 (Pin_3), R10.1
- net B2: now also U3.6 (2B); no longer J2.3 (Pin_3)
- net B3: now also U5.7 (1B); no longer J4.3 (Pin_3)
- net B4: now also U8.2 (ADC), U5.6 (2B); no longer J6.3 (Pin_3), U8.12 (GPIO10)
- net GND: now also U3.4 (GND), U5.4 (GND); no longer R10.2
- new net: R6.1, U3.5 (DIR)
- new net: R10.1, U5.5 (DIR)
- new net Button1_sense: J1.3 (Pin_3), U3.2 (1A)
- new net Button2_sense: J2.3 (Pin_3), U3.3 (2A)
- new net Button3_sense: J4.3 (Pin_3), U5.2 (1A)
- new net Button4_sense: J6.3 (Pin_3), U5.3 (2A)
